Commit message: Drop the parallel gripper from the combined model
The gripper and the adapter bolt to the same link6 flange, so a model showing
both is a model of a robot that cannot exist. Which one is present is a fact
about the robot rather than a command-line mood, so it lives in robots.yaml as
`adapter.keep_gripper: false`; --keep-gripper/--no-gripper still override it
for a one-off render. The generated URDF goes from 28 links / 27 joints to
25 / 24 -- gripper_link, gripper_left and gripper_right and their three joints.

The staleness test now compares the whole joint set, not just the two mount
origins, so a checked-in URDF that disagrees with robots.yaml about the
gripper fails the same way a moved mount does.

The studio's clankers profile gets its own joint-target normalizer: the arm02
one synthesizes gripper_joint1/2 from joint7, and while the viewer skips joints
the URDF lacks, feeding it names that cannot exist made the map lie about what
it drives.

This does not touch `arm.lerobot.use_gripper`, which is a separate decision
about how many motors the arm gateway expects.

Co-Authored-By: Claude Opus 5 <noreply@anthropic.com>

File: apps/studio/public/resources/clankers/urdf/clankers_combined.urdf (robot description, URDF)
Before this commit: robot clankers_combined, 28 links, 27 joints
Links:
- removed link gripper_left
- removed link gripper_link
- removed link gripper_right
Joints:
- removed joint gripper_joint
- removed joint gripper_joint1
- removed joint gripper_joint2

Commit message: Relabel the hand: 0-3 index, 4-7 middle, 8-11 ring, 12-15 thumb
Confirmed on hardware by jogging each group from the studio and watching which
finger moved. Only the index was labelled correctly; 4-7 were called "thumb",
8-11 "middle" and 12-15 "ring".

The old labels rested on a belief, written into the glossary, that "the LEAP
URDF's thumb_* links are actually the ring finger". They are not: the URDF's
12-15 chain is pip_4 -> thumb_pip -> thumb_dip -> thumb_fingertip, those four
joints carry limits unlike the other twelve (which is what a thumb looks like
and three identical fingers do not), and the hardware agrees with both. The
belief was the bug, and it had been propagating: docs/glossary.md asserted it,
and clankers.teleop.retarget compensated for it by mapping the human thumb onto
ring_* joints with a `thumb_gain` keyed off the "ring_" prefix.

With the labels corrected that compensation collapses: FINGER_MAP is now the
identity, human finger to robot finger of the same name. The retarget math was
physically right all along, just expressed through wrong names -- so this
changes no behaviour there, only what it is called.

Canonical indices, servo_ids and limits are untouched; they were verified
against the LEAP URDF earlier and were never in doubt. Renaming had to be one
simultaneous pass, since it is a permutation (old middle_pip -> ring_pip while
old ring_pip -> thumb_pip) that sequential replacement would corrupt.

hand.calibrated is now true, which unlocks whole-hand `pos` in the gateway, the
plugin and both studio pages. Not swept independently: the direction sign of
each individual joint -- motion looked right during the check, and travel stays
bounded by safety.max_step_rad, but one reversed joint would not have shown up.

The tests that asserted `calibrated is False` now construct an uncalibrated
config instead of reading robots.yaml, so confirming the hand cannot silently
delete the guard's coverage, and the gateway gains a test for the path this
opens. UI tests assert against the config rather than a fixed value.

Co-Authored-By: Claude Opus 5 <noreply@anthropic.com>

File: apps/studio/public/resources/clankers/urdf/clankers_combined.urdf (robot description, URDF)
Before this commit: robot clankers_combined, 25 links, 24 joints
Joints:
- removed joint ring_base_rot
- removed joint thumb_mcp_side
- added joint ring_mcp_side: type revolute, parent hand_mcp_joint_3, child hand_pip_3, origin xyz=-0.012200000000000004244 0.038100000000000001921 0.014499999999999999001 rpy=-1.570796326794896558 -1.0065212660796360242e-15 1.5707963267948943376, axis 0 0 -1, limit lower=-1.047 upper=1.047 effort=0.95 velocity=8.48
- added joint thumb_base_rot: type revolute, parent hand_palm_lower, child hand_pip_4, origin xyz=-0.069395249652862533996 -0.0012422438651005258004 -0.021622403578460215601 rpy=-8.2381766464939424156e-17 1.5707963267948956698 0, axis 0 0 -1, limit lower=-0.349 upper=2.094 effort=0.95 velocity=8.48
- joint middle_dip: child hand_fingertip_3 -> hand_fingertip_2; origin xyz=9.7144514654701197287e-17 -0.036099999999999868305 0.00020000000000007511769 rpy=4.5935029425113685044e-17 -2.8730071914463799514e-16 1.5565411607615035382e-32 -> xyz=1.0061396160665481148e-16 -0.036099999999999854428 0.00020000000000007858714 rpy=4.5935029425113654229e-17 -2.8730071914463794583e-16 1.4408183216511868558e-31; parent hand_dip_3 -> hand_dip_2
- joint middle_mcp_flex: child hand_mcp_joint_3 -> hand_mcp_joint_2; origin xyz=-0.0070952454426398371343 -0.067842243865100515521 -0.018722407666402932774 rpy=1.5707963267948950037 1.5707963267948945596 0 -> xyz=-0.0070952496528625388569 -0.022392243865100525113 -0.018722403578460229678 rpy=1.570796326794896558 1.570796326794896558 0
- joint middle_mcp_side: child hand_pip_3 -> hand_pip_2; origin xyz=-0.012200000000000004244 0.038100000000000001921 0.014499999999999999001 rpy=-1.570796326794896558 -1.0065212660796360242e-15 1.5707963267948943376 -> xyz=-0.012200000000000019856 0.038099999999999981104 0.01450000000000000594 rpy=-1.570796326794896558 -1.0065212760057939085e-15 1.5707963267948943376; parent hand_mcp_joint_3 -> hand_mcp_joint_2
- joint middle_pip: child hand_dip_3 -> hand_dip_2; origin xyz=0.014999999999999971689 0.014299999999999951639 -0.012999999999999959505 rpy=1.5707963267948958919 -1.570796326794896336 0 -> xyz=0.014999999999999975159 0.014300000000000000211 -0.013000000000000018485 rpy=1.5707963267948958919 -1.570796326794896336 0; parent hand_pip_3 -> hand_pip_2
- joint ring_dip: child hand_thumb_fingertip -> hand_fingertip_3; limit lower=-1.34 upper=1.88 effort=0.95 velocity=8.48 -> lower=-0.366 upper=2.042 effort=0.95 velocity=8.48; origin xyz=-1.249000902703301108e-16 0.046599999999999863753 0.00019999999999997710581 rpy=1.5063958491491781023e-44 5.4234187233935260503e-31 3.141592653589793116 -> xyz=9.7144514654701197287e-17 -0.036099999999999868305 0.00020000000000007511769 rpy=4.5935029425113685044e-17 -2.8730071914463799514e-16 1.5565411607615035382e-32; parent hand_thumb_dip -> hand_dip_3
- joint ring_mcp_flex: child hand_thumb_pip -> hand_mcp_joint_3; limit lower=-0.47 upper=2.443 effort=0.95 velocity=8.48 -> lower=-0.314 upper=2.23 effort=0.95 velocity=8.48; origin xyz=-2.7755575615628913511e-17 0.014300000000000005415 -0.013000000000000011546 rpy=1.5707963267948958919 -1.570796326794896336 0 -> xyz=-0.0070952454426398371343 -0.067842243865100515521 -0.018722407666402932774 rpy=1.5707963267948950037 1.5707963267948945596 0; parent hand_pip_4 -> hand_palm_lower
- joint ring_pip: child hand_thumb_dip -> hand_dip_3; limit lower=-1.20 upper=1.90 effort=0.95 velocity=8.48 -> lower=-0.506 upper=1.885 effort=0.95 velocity=8.48; origin xyz=0 0.014499999999999966041 -0.017000000000000053263 rpy=-1.570796326794896558 1.6050198443300131245e-46 -1.9721522630516624601e-31 -> xyz=0.014999999999999971689 0.014299999999999951639 -0.012999999999999959505 rpy=1.5707963267948958919 -1.570796326794896336 0; parent hand_thumb_pip -> hand_pip_3
- joint thumb_dip: child hand_fingertip_2 -> hand_thumb_fingertip; limit lower=-0.366 upper=2.042 effort=0.95 velocity=8.48 -> lower=-1.34 upper=1.88 effort=0.95 velocity=8.48; origin xyz=1.0061396160665481148e-16 -0.036099999999999854428 0.00020000000000007858714 rpy=4.5935029425113654229e-17 -2.8730071914463794583e-16 1.4408183216511868558e-31 -> xyz=-1.249000902703301108e-16 0.046599999999999863753 0.00019999999999997710581 rpy=1.5063958491491781023e-44 5.4234187233935260503e-31 3.141592653589793116; parent hand_dip_2 -> hand_thumb_dip
- joint thumb_mcp_flex: child hand_mcp_joint_2 -> hand_thumb_pip; limit lower=-0.314 upper=2.23 effort=0.95 velocity=8.48 -> lower=-0.47 upper=2.443 effort=0.95 velocity=8.48; origin xyz=-0.0070952496528625388569 -0.022392243865100525113 -0.018722403578460229678 rpy=1.570796326794896558 1.570796326794896558 0 -> xyz=-2.7755575615628913511e-17 0.014300000000000005415 -0.013000000000000011546 rpy=1.5707963267948958919 -1.570796326794896336 0; parent hand_palm_lower -> hand_pip_4
- joint thumb_pip: child hand_dip_2 -> hand_thumb_dip; limit lower=-0.506 upper=1.885 effort=0.95 velocity=8.48 -> lower=-1.20 upper=1.90 effort=0.95 velocity=8.48; origin xyz=0.014999999999999975159 0.014300000000000000211 -0.013000000000000018485 rpy=1.5707963267948958919 -1.570796326794896336 0 -> xyz=0 0.014499999999999966041 -0.017000000000000053263 rpy=-1.570796326794896558 1.6050198443300131245e-46 -1.9721522630516624601e-31; parent hand_pip_2 -> hand_thumb_pip
